Commit message: feat(sim): 接入 gz sim 主线并冻结复用边界
- 新增 simulation.launch.py、simulation.yaml 和基础 world，建立 gz sim + ros2_control + MoveIt 的仿真启动链\n- 扩展 URDF/ros2_control xacro，支持仿真 backend 注入并补齐关节速度/力矩限制\n- 更新项目与 P4 文档，明确任务层/合同层复用、backend 层分叉，以及当前主开发环境切到仿真

File: src/dual_nero_description/urdf/nero_single_arm_macro.xacro (robot description, xacro)
@@ -46,5 +46,5 @@
       <child link="${prefix}link1"/>
       <axis xyz="0 0 1"/>
-      <limit lower="-2.7" upper="2.7" effort="0" velocity="0"/>
+      <limit lower="-2.7" upper="2.7" effort="50" velocity="1.0"/>
     </joint>
     <link name="${prefix}link2">
@@ -62,5 +62,5 @@
       <child link="${prefix}link2"/>
       <axis xyz="0 0 1"/>
-      <limit lower="-1.74" upper="1.74" effort="0" velocity="0"/>
+      <limit lower="-1.74" upper="1.74" effort="50" velocity="1.0"/>
     </joint>
     <link name="${prefix}link3">
@@ -78,5 +78,5 @@
       <child link="${prefix}link3"/>
       <axis xyz="0 0 1"/>
-      <limit lower="-2.75" upper="2.75" effort="0" velocity="0"/>
+      <limit lower="-2.75" upper="2.75" effort="50" velocity="1.0"/>
     </joint>
     <link name="${prefix}link4">
@@ -94,5 +94,5 @@
       <child link="${prefix}link4"/>
       <axis xyz="0 0 1"/>
-      <limit lower="-1.01" upper="2.14" effort="0" velocity="0"/>
+      <limit lower="-1.01" upper="2.14" effort="50" velocity="1.0"/>
     </joint>
     <link name="${prefix}link5">
@@ -110,5 +110,5 @@
       <child link="${prefix}link5"/>
       <axis xyz="0 0 1"/>
-      <limit lower="-2.75" upper="2.75" effort="0" velocity="0"/>
+      <limit lower="-2.75" upper="2.75" effort="50" velocity="1.0"/>
     </joint>
     <link name="${prefix}link6">
@@ -126,5 +126,5 @@
       <child link="${prefix}link6"/>
       <axis xyz="0 0 1"/>
-      <limit lower="-0.73" upper="0.95" effort="0" velocity="0"/>
+      <limit lower="-0.73" upper="0.95" effort="50" velocity="1.0"/>
     </joint>
     <link name="${prefix}link7">
@@ -142,5 +142,5 @@
       <child link="${prefix}link7"/>
       <axis xyz="0 0 1"/>
-      <limit lower="-1.57" upper="1.57" effort="0" velocity="0"/>
+      <limit lower="-1.57" upper="1.57" effort="50" velocity="1.0"/>
     </joint>
     <link name="${prefix}end_effector">

File: src/dual_nero_moveit_config/config/dual_nero_description.ros2_control.xacro (robot description, xacro)
@@ -1,10 +1,12 @@
 <?xml version="1.0"?>
 <robot xmlns:xacro="http://www.ros.org/wiki/xacro">
-    <xacro:macro name="dual_nero_description_ros2_control" params="name initial_positions_file">
+    <xacro:macro
+        name="dual_nero_description_ros2_control"
+        params="name initial_positions_file hardware_plugin:='mock_components/GenericSystem' use_gz_sim:='false' controllers_file:=''"
+    >
         <xacro:property name="initial_positions" value="${load_yaml(initial_positions_file)['initial_positions']}"/>
         <ros2_control name="${name}" type="system">
             <hardware>
-                <!-- By default, set up controllers for simulation. This won't work on real hardware -->
-                <plugin>mock_components/GenericSystem</plugin>
+                <plugin>${hardware_plugin}</plugin>
             </hardware>
             <joint name="left_joint1">
@@ -107,4 +109,11 @@
             </joint>
         </ros2_control>
+        <xacro:if value="${use_gz_sim == 'true'}">
+            <gazebo>
+                <plugin filename="libgz_ros2_control-system.so" name="gz_ros2_control::GazeboSimROS2ControlPlugin">
+                    <parameters>${controllers_file}</parameters>
+                </plugin>
+            </gazebo>
+        </xacro:if>
     </xacro:macro>
 </robot>

File: src/dual_nero_moveit_config/config/dual_nero_description.urdf.xacro (robot description, xacro)
@@ -2,8 +2,17 @@
 <robot xmlns:xacro="http://www.ros.org/wiki/xacro" name="dual_nero_description">
     <xacro:arg name="initial_positions_file" default="initial_positions.yaml" />
+    <xacro:arg name="hardware_plugin" default="mock_components/GenericSystem" />
+    <xacro:arg name="use_gz_sim" default="false" />
+    <xacro:arg name="controllers_file" default="" />
     <!-- Import dual_nero_description urdf file -->
     <xacro:include filename="$(find dual_nero_description)/urdf/dual_nero_description.xacro" />
     <!-- Import control_xacro -->
     <xacro:include filename="dual_nero_description.ros2_control.xacro" />
-    <xacro:dual_nero_description_ros2_control name="FakeSystem" initial_positions_file="$(arg initial_positions_file)"/>
+    <xacro:dual_nero_description_ros2_control
+        name="FakeSystem"
+        initial_positions_file="$(arg initial_positions_file)"
+        hardware_plugin="$(arg hardware_plugin)"
+        use_gz_sim="$(arg use_gz_sim)"
+        controllers_file="$(arg controllers_file)"
+    />
 </robot>

Commit message: fix(sim): 兼容布尔型仿真 visual 开关判断
- 将 use_sim_visuals 的 xacro 判断改为对字符串/布尔都稳的形式\n- 确保 use_gz_sim=true 时生成 STL visual mesh 而不是继续回退到 DAE\n- 为 Gazebo 仿真摆脱 DAE 渲染链问题提供最终参数修正

File: src/dual_nero_description/urdf/nero_single_arm_macro.xacro (robot description, xacro)
@@ -8,13 +8,14 @@
   -->
   <xacro:macro name="nero_single_arm" params="prefix parent xyz:='0 0 0' rpy:='0 0 0' use_sim_visuals:='false'">
-    <xacro:property name="base_visual_mesh" value="${'package://dual_nero_description/meshes/base_link.STL' if use_sim_visuals == 'true' else 'package://dual_nero_description/meshes/dae/base_link.dae'}"/>
-    <xacro:property name="link1_visual_mesh" value="${'package://dual_nero_description/meshes/Link1.STL' if use_sim_visuals == 'true' else 'package://dual_nero_description/meshes/dae/link1.dae'}"/>
-    <xacro:property name="link2_visual_mesh" value="${'package://dual_nero_description/meshes/Link2.STL' if use_sim_visuals == 'true' else 'package://dual_nero_description/meshes/dae/link2.dae'}"/>
-    <xacro:property name="link3_visual_mesh" value="${'package://dual_nero_description/meshes/Link3.STL' if use_sim_visuals == 'true' else 'package://dual_nero_description/meshes/dae/link3.dae'}"/>
-    <xacro:property name="link4_visual_mesh" value="${'package://dual_nero_description/meshes/Link4.STL' if use_sim_visuals == 'true' else 'package://dual_nero_description/meshes/dae/link4.dae'}"/>
-    <xacro:property name="link5_visual_mesh" value="${'package://dual_nero_description/meshes/Link5.STL' if use_sim_visuals == 'true' else 'package://dual_nero_description/meshes/dae/link5.dae'}"/>
-    <xacro:property name="link6_visual_mesh" value="${'package://dual_nero_description/meshes/Link6.STL' if use_sim_visuals == 'true' else 'package://dual_nero_description/meshes/dae/link6.dae'}"/>
-    <xacro:property name="link7_visual_mesh" value="${'package://dual_nero_description/meshes/Link7.STL' if use_sim_visuals == 'true' else 'package://dual_nero_description/meshes/dae/link7.dae'}"/>
-    <xacro:property name="ee_visual_mesh" value="${'package://dual_nero_description/meshes/stand_v2.STL' if use_sim_visuals == 'true' else 'package://dual_nero_description/meshes/stand_v1.dae'}"/>
+    <xacro:property name="sim_visuals_enabled" value="${str(use_sim_visuals).lower() == 'true'}"/>
+    <xacro:property name="base_visual_mesh" value="${'package://dual_nero_description/meshes/base_link.STL' if sim_visuals_enabled else 'package://dual_nero_description/meshes/dae/base_link.dae'}"/>
+    <xacro:property name="link1_visual_mesh" value="${'package://dual_nero_description/meshes/Link1.STL' if sim_visuals_enabled else 'package://dual_nero_description/meshes/dae/link1.dae'}"/>
+    <xacro:property name="link2_visual_mesh" value="${'package://dual_nero_description/meshes/Link2.STL' if sim_visuals_enabled else 'package://dual_nero_description/meshes/dae/link2.dae'}"/>
+    <xacro:property name="link3_visual_mesh" value="${'package://dual_nero_description/meshes/Link3.STL' if sim_visuals_enabled else 'package://dual_nero_description/meshes/dae/link3.dae'}"/>
+    <xacro:property name="link4_visual_mesh" value="${'package://dual_nero_description/meshes/Link4.STL' if sim_visuals_enabled else 'package://dual_nero_description/meshes/dae/link4.dae'}"/>
+    <xacro:property name="link5_visual_mesh" value="${'package://dual_nero_description/meshes/Link5.STL' if sim_visuals_enabled else 'package://dual_nero_description/meshes/dae/link5.dae'}"/>
+    <xacro:property name="link6_visual_mesh" value="${'package://dual_nero_description/meshes/Link6.STL' if sim_visuals_enabled else 'package://dual_nero_description/meshes/dae/link6.dae'}"/>
+    <xacro:property name="link7_visual_mesh" value="${'package://dual_nero_description/meshes/Link7.STL' if sim_visuals_enabled else 'package://dual_nero_description/meshes/dae/link7.dae'}"/>
+    <xacro:property name="ee_visual_mesh" value="${'package://dual_nero_description/meshes/stand_v2.STL' if sim_visuals_enabled else 'package://dual_nero_description/meshes/stand_v1.dae'}"/>
     <link name="${prefix}base_link">
       <inertial>
@@ -165,5 +166,5 @@
       <collision>
         <origin xyz="0 0 0" rpy="-1.57 -1.57 -1.57"/>
-        <geometry><mesh filename="${'package://dual_nero_description/meshes/stand_v2.STL' if use_sim_visuals == 'true' else 'package://dual_nero_description/meshes/stand_v1.dae'}"/></geometry>
+        <geometry><mesh filename="${'package://dual_nero_description/meshes/stand_v2.STL' if sim_visuals_enabled else 'package://dual_nero_description/meshes/stand_v1.dae'}"/></geometry>
       </collision>
     </link>
