Commit message: fix(sim): 仿真时切换 STL visual mesh 规避 Gazebo Ogre2 崩溃
- 为单臂 xacro 增加 use_sim_visuals 开关，仿真时使用 STL 作为 visual mesh\n- 保留非仿真场景下的 DAE 视觉资产，不影响现有 MoveIt/RViz 语义\n- 解决 Gazebo Harmonic 加载双臂 DAE 时触发 UV 通道断言并导致 controller 链无法启动的问题

File: src/dual_nero_description/urdf/dual_nero_description.xacro (robot description, xacro)
@@ -1,4 +1,5 @@
 <?xml version="1.0"?>
 <robot name="dual_nero_description" xmlns:xacro="http://www.ros.org/wiki/xacro">
+  <xacro:arg name="use_sim_visuals" default="false"/>
   <!-- 引入单臂宏 -->
   <xacro:include filename="$(find dual_nero_description)/urdf/nero_single_arm_macro.xacro"/>
@@ -83,5 +84,6 @@
       parent="dual_crossbar"
       xyz="-0.145 0 0"
-      rpy="0 -1.5708 0"/>
+      rpy="0 -1.5708 0"
+      use_sim_visuals="$(arg use_sim_visuals)"/>
   <!-- 左臂 -->
   <xacro:nero_single_arm
@@ -89,4 +91,5 @@
       parent="dual_crossbar"
       xyz="0.145 0 0"
-      rpy="0 -1.5708 3.14159"/>
+      rpy="0 -1.5708 3.14159"
+      use_sim_visuals="$(arg use_sim_visuals)"/>
 </robot>

File: src/dual_nero_description/urdf/nero_single_arm_macro.xacro (robot description, xacro)
@@ -7,5 +7,14 @@
     xyz/rpy:   arm mount pose relative to parent
   -->
-  <xacro:macro name="nero_single_arm" params="prefix parent xyz:='0 0 0' rpy:='0 0 0'">
+  <xacro:macro name="nero_single_arm" params="prefix parent xyz:='0 0 0' rpy:='0 0 0' use_sim_visuals:='false'">
+    <xacro:property name="base_visual_mesh" value="${'package://dual_nero_description/meshes/base_link.STL' if use_sim_visuals == 'true' else 'package://dual_nero_description/meshes/dae/base_link.dae'}"/>
+    <xacro:property name="link1_visual_mesh" value="${'package://dual_nero_description/meshes/Link1.STL' if use_sim_visuals == 'true' else 'package://dual_nero_description/meshes/dae/link1.dae'}"/>
+    <xacro:property name="link2_visual_mesh" value="${'package://dual_nero_description/meshes/Link2.STL' if use_sim_visuals == 'true' else 'package://dual_nero_description/meshes/dae/link2.dae'}"/>
+    <xacro:property name="link3_visual_mesh" value="${'package://dual_nero_description/meshes/Link3.STL' if use_sim_visuals == 'true' else 'package://dual_nero_description/meshes/dae/link3.dae'}"/>
+    <xacro:property name="link4_visual_mesh" value="${'package://dual_nero_description/meshes/Link4.STL' if use_sim_visuals == 'true' else 'package://dual_nero_description/meshes/dae/link4.dae'}"/>
+    <xacro:property name="link5_visual_mesh" value="${'package://dual_nero_description/meshes/Link5.STL' if use_sim_visuals == 'true' else 'package://dual_nero_description/meshes/dae/link5.dae'}"/>
+    <xacro:property name="link6_visual_mesh" value="${'package://dual_nero_description/meshes/Link6.STL' if use_sim_visuals == 'true' else 'package://dual_nero_description/meshes/dae/link6.dae'}"/>
+    <xacro:property name="link7_visual_mesh" value="${'package://dual_nero_description/meshes/Link7.STL' if use_sim_visuals == 'true' else 'package://dual_nero_description/meshes/dae/link7.dae'}"/>
+    <xacro:property name="ee_visual_mesh" value="${'package://dual_nero_description/meshes/stand_v2.STL' if use_sim_visuals == 'true' else 'package://dual_nero_description/meshes/stand_v1.dae'}"/>
     <link name="${prefix}base_link">
       <inertial>
@@ -17,5 +26,5 @@
         <origin xyz="0 0 0" rpy="0 0 0"/>
         <geometry>
-          <mesh filename="package://dual_nero_description/meshes/dae/base_link.dae"/>
+          <mesh filename="${base_visual_mesh}"/>
         </geometry>
       </visual>
@@ -38,5 +47,5 @@
         <inertia ixx="0.0006669" ixy="0.0" ixz="0.0" iyy="0.00054501" iyz="0.0" izz="0.00051509"/>
       </inertial>
-      <visual><origin xyz="0 0 0" rpy="0 0 0"/><geometry><mesh filename="package://dual_nero_description/meshes/dae/link1.dae"/></geometry></visual>
+      <visual><origin xyz="0 0 0" rpy="0 0 0"/><geometry><mesh filename="${link1_visual_mesh}"/></geometry></visual>
       <collision><origin xyz="0 0 0" rpy="0 0 0"/><geometry><mesh filename="package://dual_nero_description/meshes/Link1.STL"/></geometry></collision>
     </link>
@@ -54,5 +63,5 @@
         <inertia ixx="0.00053808" ixy="0.0" ixz="0.0" iyy="0.00029435" iyz="0.0" izz="0.00040266"/>
       </inertial>
-      <visual><origin xyz="0 0 0" rpy="0 0 0"/><geometry><mesh filename="package://dual_nero_description/meshes/dae/link2.dae"/></geometry></visual>
+      <visual><origin xyz="0 0 0" rpy="0 0 0"/><geometry><mesh filename="${link2_visual_mesh}"/></geometry></visual>
       <collision><origin xyz="0 0 0" rpy="0 0 0"/><geometry><mesh filename="package://dual_nero_description/meshes/Link2.STL"/></geometry></collision>
     </link>
@@ -70,5 +79,5 @@
         <inertia ixx="0.00342528" ixy="0.0" ixz="0.0" iyy="0.0033924" iyz="0.0" izz="0.00026169"/>
       </inertial>
-      <visual><origin xyz="0 0 0" rpy="0 0 0"/><geometry><mesh filename="package://dual_nero_description/meshes/dae/link3.dae"/></geometry></visual>
+      <visual><origin xyz="0 0 0" rpy="0 0 0"/><geometry><mesh filename="${link3_visual_mesh}"/></geometry></visual>
       <collision><origin xyz="0 0 0" rpy="0 0 0"/><geometry><mesh filename="package://dual_nero_description/meshes/Link3.STL"/></geometry></collision>
     </link>
@@ -86,5 +95,5 @@
         <inertia ixx="0.00031331" ixy="0.0" ixz="0.0" iyy="0.00013204" iyz="0.0" izz="0.0002393"/>
       </inertial>
-      <visual><origin xyz="0 0 0" rpy="0 0 0"/><geometry><mesh filename="package://dual_nero_description/meshes/dae/link4.dae"/></geometry></visual>
+      <visual><origin xyz="0 0 0" rpy="0 0 0"/><geometry><mesh filename="${link4_visual_mesh}"/></geometry></visual>
       <collision><origin xyz="0 0 0" rpy="0 0 0"/><geometry><mesh filename="package://dual_nero_description/meshes/Link4.STL"/></geometry></collision>
     </link>
@@ -102,5 +111,5 @@
         <inertia ixx="0.0008249" ixy="0.0" ixz="0.0" iyy="0.00078548" iyz="0.0" izz="0.00021015"/>
       </inertial>
-      <visual><origin xyz="0 0 0" rpy="0 0 0"/><geometry><mesh filename="package://dual_nero_description/meshes/dae/link5.dae"/></geometry></visual>
+      <visual><origin xyz="0 0 0" rpy="0 0 0"/><geometry><mesh filename="${link5_visual_mesh}"/></geometry></visual>
       <collision><origin xyz="0 0 0" rpy="0 0 0"/><geometry><mesh filename="package://dual_nero_description/meshes/Link5.STL"/></geometry></collision>
     </link>
@@ -118,5 +127,5 @@
         <inertia ixx="0.00008181" ixy="0.0" ixz="0.0" iyy="0.00007176" iyz="0.0" izz="0.00007906"/>
       </inertial>
-      <visual><origin xyz="0 0 0" rpy="0 0 0"/><geometry><mesh filename="package://dual_nero_description/meshes/dae/link6.dae"/></geometry></visual>
+      <visual><origin xyz="0 0 0" rpy="0 0 0"/><geometry><mesh filename="${link6_visual_mesh}"/></geometry></visual>
       <collision><origin xyz="0 0 0" rpy="0 0 0"/><geometry><mesh filename="package://dual_nero_description/meshes/Link6.STL"/></geometry></collision>
     </link>
@@ -134,5 +143,5 @@
         <inertia ixx="1.1000000000000001e-07" ixy="0" ixz="0" iyy="1.1000000000000001e-07" iyz="0" izz="1.9999999999999999e-07"/>
       </inertial>
-      <visual><origin xyz="0 0 0" rpy="0 0 0"/><geometry><mesh filename="package://dual_nero_description/meshes/dae/link7.dae"/></geometry></visual>
+      <visual><origin xyz="0 0 0" rpy="0 0 0"/><geometry><mesh filename="${link7_visual_mesh}"/></geometry></visual>
       <collision><origin xyz="0 0 0" rpy="0 0 0"/><geometry><mesh filename="package://dual_nero_description/meshes/Link7.STL"/></geometry></collision>
     </link>
@@ -152,9 +161,9 @@
       <visual>
         <origin xyz="0 0 0" rpy="-1.57 -1.57 -1.57"/>
-        <geometry><mesh filename="package://dual_nero_description/meshes/stand_v1.dae"/></geometry>
+        <geometry><mesh filename="${ee_visual_mesh}"/></geometry>
       </visual>
       <collision>
         <origin xyz="0 0 0" rpy="-1.57 -1.57 -1.57"/>
-        <geometry><mesh filename="package://dual_nero_description/meshes/stand_v1.dae"/></geometry>
+        <geometry><mesh filename="${'package://dual_nero_description/meshes/stand_v2.STL' if use_sim_visuals == 'true' else 'package://dual_nero_description/meshes/stand_v1.dae'}"/></geometry>
       </collision>
     </link>

File: src/dual_nero_moveit_config/config/dual_nero_description.urdf.xacro (robot description, xacro)
@@ -5,4 +5,5 @@
     <xacro:arg name="use_gz_sim" default="false" />
     <xacro:arg name="controllers_file" default="" />
+    <xacro:arg name="use_sim_visuals" default="$(arg use_gz_sim)" />
     <!-- Import dual_nero_description urdf file -->
     <xacro:include filename="$(find dual_nero_description)/urdf/dual_nero_description.xacro" />

Commit message: fix(sim): 修正仿真 visual mesh 开关传递链
- 将 use_sim_visuals 从顶层 urdf xacro 正确传递到双臂描述 xacro\n- 确保 use_gz_sim=true 时生成 STL visual mesh 而不是 DAE\n- 为 Gazebo Harmonic 下双臂模型稳定显示和后续控制器链恢复提供前提

File: src/dual_nero_description/urdf/dual_nero_description.xacro (robot description, xacro)
@@ -1,5 +1,4 @@
 <?xml version="1.0"?>
 <robot name="dual_nero_description" xmlns:xacro="http://www.ros.org/wiki/xacro">
-  <xacro:arg name="use_sim_visuals" default="false"/>
   <!-- 引入单臂宏 -->
   <xacro:include filename="$(find dual_nero_description)/urdf/nero_single_arm_macro.xacro"/>
@@ -85,5 +84,5 @@
       xyz="-0.145 0 0"
       rpy="0 -1.5708 0"
-      use_sim_visuals="$(arg use_sim_visuals)"/>
+      use_sim_visuals="${use_sim_visuals}"/>
   <!-- 左臂 -->
   <xacro:nero_single_arm
@@ -92,4 +91,4 @@
       xyz="0.145 0 0"
       rpy="0 -1.5708 3.14159"
-      use_sim_visuals="$(arg use_sim_visuals)"/>
+      use_sim_visuals="${use_sim_visuals}"/>
 </robot>

File: src/dual_nero_moveit_config/config/dual_nero_description.urdf.xacro (robot description, xacro)
@@ -7,4 +7,5 @@
     <xacro:arg name="use_sim_visuals" default="$(arg use_gz_sim)" />
     <!-- Import dual_nero_description urdf file -->
+    <xacro:property name="use_sim_visuals" value="$(arg use_sim_visuals)" />
     <xacro:include filename="$(find dual_nero_description)/urdf/dual_nero_description.xacro" />
     <!-- Import control_xacro -->

Commit message: refactor(urdf): 参数化双臂公共安装结构
- 保持单臂宏不变，只重构双臂公共安装结构
- 将支撑框、横杆、左右安装盒和挂载位抽成正式参数
- 按第一轮实测值更新默认结构尺寸
- 新增安装结构参数文档，并明确待校正的 mount pose 项

File: src/dual_nero_description/urdf/dual_nero_description.xacro (robot description, xacro)
@@ -1,7 +1,39 @@
 <?xml version="1.0"?>
 <robot name="dual_nero_description" xmlns:xacro="http://www.ros.org/wiki/xacro">
-  <!-- 引入单臂宏 -->
+  <xacro:arg name="use_sim_visuals" default="false"/>
+  <xacro:arg name="world_to_base_xyz" default="0 0 0"/>
+  <xacro:arg name="world_to_base_rpy" default="0 0 0"/>
+  <xacro:arg name="base_plate_size" default="0.20 0.08 0.04"/>
+  <xacro:arg name="base_plate_visual_xyz" default="0 0 0.02"/>
+  <xacro:arg name="column_size" default="0.04 0.04 1.50"/>
+  <xacro:arg name="column_visual_xyz" default="0 0 0.75"/>
+  <xacro:arg name="column_joint_xyz" default="0 0 0.04"/>
+  <xacro:arg name="column_joint_rpy" default="0 0 0"/>
+  <xacro:arg name="enable_support_frame" default="true"/>
+  <xacro:arg name="support_frame_size" default="0.23 0.01 0.30"/>
+  <xacro:arg name="support_frame_visual_xyz" default="0 0 0.15"/>
+  <xacro:arg name="support_frame_joint_xyz" default="0 0.06 0.49"/>
+  <xacro:arg name="support_frame_joint_rpy" default="0 0 0"/>
+  <xacro:arg name="crossbar_size" default="0.25 0.04 0.04"/>
+  <xacro:arg name="crossbar_joint_xyz" default="0 0 0.81"/>
+  <xacro:arg name="crossbar_joint_rpy" default="0 0 0"/>
+  <xacro:arg name="left_mount_box_size" default="0.07 0.02 0.095"/>
+  <xacro:arg name="left_mount_box_xyz" default="0.13 0 0"/>
+  <xacro:arg name="left_mount_box_rpy" default="0 0 0"/>
+  <xacro:arg name="right_mount_box_size" default="0.07 0.02 0.095"/>
+  <xacro:arg name="right_mount_box_xyz" default="-0.13 0 0"/>
+  <xacro:arg name="right_mount_box_rpy" default="0 0 0"/>
+  <xacro:arg name="left_mount_xyz" default="0 0 0"/>
+  <xacro:arg name="left_mount_rpy" default="0 -1.5708 3.14159"/>
+  <xacro:arg name="right_mount_xyz" default="0 0 0"/>
+  <xacro:arg name="right_mount_rpy" default="0 -1.5708 0"/>
+  <xacro:property name="support_frame_enabled" value="${str(enable_support_frame).lower() == 'true'}"/>
+  <!--
+    Reuse the validated single-arm chain and only parameterize the shared mount structure.
+    Length values are in meters. The current defaults come from the 2026-04-23 first-pass
+    measurement set and intentionally keep arm mount offsets at zero relative to each mount box
+    until the physical mounting-face center and orientation are re-measured.
+  -->
   <xacro:include filename="$(find dual_nero_description)/urdf/nero_single_arm_macro.xacro"/>
-  <!-- 颜色材质 -->
   <material name="blue">
     <color rgba="0.2 0.4 0.9 1.0"/>
@@ -13,19 +45,17 @@
     <color rgba="0.8 0.8 0.8 1.0"/>
   </material>
-  <!-- 世界坐标 -->
   <link name="world"/>
-  <!-- 底座 -->
   <link name="dual_base_plate">
     <visual>
-      <origin xyz="0 0 0.02" rpy="0 0 0"/>
+      <origin xyz="$(arg base_plate_visual_xyz)" rpy="0 0 0"/>
       <geometry>
-        <box size="0.20 0.08 0.04"/>
+        <box size="$(arg base_plate_size)"/>
       </geometry>
       <material name="blue"/>
     </visual>
     <collision>
-      <origin xyz="0 0 0.02" rpy="0 0 0"/>
+      <origin xyz="$(arg base_plate_visual_xyz)" rpy="0 0 0"/>
       <geometry>
-        <box size="0.20 0.08 0.04"/>
+        <box size="$(arg base_plate_size)"/>
       </geometry>
     </collision>
@@ -34,19 +64,18 @@
     <parent link="world"/>
     <child link="dual_base_plate"/>
-    <origin xyz="0 0 0" rpy="0 0 0"/>
+    <origin xyz="$(arg world_to_base_xyz)" rpy="$(arg world_to_base_rpy)"/>
   </joint>
-  <!-- 立柱 -->
   <link name="dual_column">
     <visual>
-      <origin xyz="0 0 0.75" rpy="0 0 0"/>
+      <origin xyz="$(arg column_visual_xyz)" rpy="0 0 0"/>
       <geometry>
-        <box size="0.04 0.04 1.50"/>
+        <box size="$(arg column_size)"/>
       </geometry>
       <material name="gray"/>
     </visual>
     <collision>
-      <origin xyz="0 0 0.75" rpy="0 0 0"/>
+      <origin xyz="$(arg column_visual_xyz)" rpy="0 0 0"/>
       <geometry>
-        <box size="0.04 0.04 1.50"/>
+        <box size="$(arg column_size)"/>
       </geometry>
     </collision>
@@ -55,12 +84,33 @@
     <parent link="dual_base_plate"/>
     <child link="dual_column"/>
-    <origin xyz="0 0 0.04" rpy="0 0 0"/>
+    <origin xyz="$(arg column_joint_xyz)" rpy="$(arg column_joint_rpy)"/>
   </joint>
-  <!-- 横梁 -->
+  <xacro:if value="${support_frame_enabled}">
+    <link name="dual_support_frame">
+      <visual>
+        <origin xyz="$(arg support_frame_visual_xyz)" rpy="0 0 0"/>
+        <geometry>
+          <box size="$(arg support_frame_size)"/>
+        </geometry>
+        <material name="gray"/>
+      </visual>
+      <collision>
+        <origin xyz="$(arg support_frame_visual_xyz)" rpy="0 0 0"/>
+        <geometry>
+          <box size="$(arg support_frame_size)"/>
+        </geometry>
+      </collision>
+    </link>
+    <joint name="dual_column_to_support_frame" type="fixed">
+      <parent link="dual_column"/>
+      <child link="dual_support_frame"/>
+      <origin xyz="$(arg support_frame_joint_xyz)" rpy="$(arg support_frame_joint_rpy)"/>
+    </joint>
+  </xacro:if>
   <link name="dual_crossbar">
     <visual>
       <origin xyz="0 0 0" rpy="0 0 0"/>
       <geometry>
-        <box size="0.34 0.05 0.05"/>
+        <box size="$(arg crossbar_size)"/>
       </geometry>
       <material name="silver"/>
@@ -69,5 +119,5 @@
       <origin xyz="0 0 0" rpy="0 0 0"/>
       <geometry>
-        <box size="0.34 0.05 0.05"/>
+        <box size="$(arg crossbar_size)"/>
       </geometry>
     </collision>
@@ -76,19 +126,57 @@
     <parent link="dual_column"/>
     <child link="dual_crossbar"/>
-    <origin xyz="0 0 1.50" rpy="0 0 0"/>
+    <origin xyz="$(arg crossbar_joint_xyz)" rpy="$(arg crossbar_joint_rpy)"/>
   </joint>
-  <!-- 右臂 -->
+  <link name="left_mount_box">
+    <visual>
+      <origin xyz="0 0 0" rpy="0 0 0"/>
+      <geometry>
+        <box size="$(arg left_mount_box_size)"/>
+      </geometry>
+      <material name="silver"/>
+    </visual>
+    <collision>
+      <origin xyz="0 0 0" rpy="0 0 0"/>
+      <geometry>
+        <box size="$(arg left_mount_box_size)"/>
+      </geometry>
+    </collision>
+  </link>
+  <joint name="dual_crossbar_to_left_mount_box" type="fixed">
+    <parent link="dual_crossbar"/>
+    <child link="left_mount_box"/>
+    <origin xyz="$(arg left_mount_box_xyz)" rpy="$(arg left_mount_box_rpy)"/>
+  </joint>
+  <link name="right_mount_box">
+    <visual>
+      <origin xyz="0 0 0" rpy="0 0 0"/>
+      <geometry>
+        <box size="$(arg right_mount_box_size)"/>
+      </geometry>
+      <material name="silver"/>
+    </visual>
+    <collision>
+      <origin xyz="0 0 0" rpy="0 0 0"/>
+      <geometry>
+        <box size="$(arg right_mount_box_size)"/>
+      </geometry>
+    </collision>
+  </link>
+  <joint name="dual_crossbar_to_right_mount_box" type="fixed">
+    <parent link="dual_crossbar"/>
+    <child link="right_mount_box"/>
+    <origin xyz="$(arg right_mount_box_xyz)" rpy="$(arg right_mount_box_rpy)"/>
+  </joint>
   <xacro:nero_single_arm
       prefix="right_"
-      parent="dual_crossbar"
-      xyz="-0.145 0 0"
-      rpy="0 -1.5708 0"
+      parent="right_mount_box"
+      xyz="$(arg right_mount_xyz)"
+      rpy="$(arg right_mount_rpy)"
       use_sim_visuals="${use_sim_visuals}"/>
-  <!-- 左臂 -->
   <xacro:nero_single_arm
       prefix="left_"
-      parent="dual_crossbar"
-      xyz="0.145 0 0"
-      rpy="0 -1.5708 3.14159"
+      parent="left_mount_box"
+      xyz="$(arg left_mount_xyz)"
+      rpy="$(arg left_mount_rpy)"
       use_sim_visuals="${use_sim_visuals}"/>
 </robot>

Commit message: fix(urdf): 修正 support frame 的 xacro 条件判断
- 去掉对 enable_support_frame 的错误表达式求值
- 直接使用 xacro arg 控制 support frame 是否生成
- 恢复 dual_nero_description.xacro 的直接展开能力

File: src/dual_nero_description/urdf/dual_nero_description.xacro (robot description, xacro)
@@ -28,5 +28,4 @@
   <xacro:arg name="right_mount_xyz" default="0 0 0"/>
   <xacro:arg name="right_mount_rpy" default="0 -1.5708 0"/>
-  <xacro:property name="support_frame_enabled" value="${str(enable_support_frame).lower() == 'true'}"/>
   <!--
     Reuse the validated single-arm chain and only parameterize the shared mount structure.
@@ -86,5 +85,5 @@
     <origin xyz="$(arg column_joint_xyz)" rpy="$(arg column_joint_rpy)"/>
   </joint>
-  <xacro:if value="${support_frame_enabled}">
+  <xacro:if value="$(arg enable_support_frame)">
     <link name="dual_support_frame">
       <visual>
