Commit message: feat(urdf): 为独立立柱模型添加顶部梯形实体
- 在 column-only 独立模型上新增上宽下窄的顶部实体
- 保持实体厚度沿 Y 方向，并使其中心线与立柱中心线重合
- 先用简化近似结构验证几何关系，为后续细化梯形轮廓做准备

File: src/dual_nero_description/urdf/dual_nero_column_only.xacro (robot description, xacro)
@@ -5,6 +5,14 @@
   <xacro:arg name="column_size" default="0.105 0.105 0.52"/>
   <xacro:arg name="column_visual_xyz" default="0 0 0.26"/>
+  <xacro:arg name="head_upper_width" default="0.25"/>
+  <xacro:arg name="head_lower_width" default="0.125"/>
+  <xacro:arg name="head_depth" default="0.125"/>
+  <xacro:arg name="head_height" default="0.31"/>
+  <xacro:arg name="head_base_xyz" default="0 0 0.52"/>
   <material name="column_silver">
     <color rgba="0.8 0.8 0.8 1.0"/>
+  </material>
+  <material name="head_gray">
+    <color rgba="0.72 0.72 0.72 1.0"/>
   </material>
   <link name="world"/>
@@ -29,3 +37,30 @@
     <origin xyz="$(arg world_to_column_xyz)" rpy="$(arg world_to_column_rpy)"/>
   </joint>
+  <link name="column_head">
+    <visual>
+      <origin xyz="0 0 0.0775" rpy="0 0 0"/>
+      <geometry>
+        <box size="0.15625 $(arg head_depth) 0.155"/>
+      </geometry>
+      <material name="head_gray"/>
+    </visual>
+    <visual>
+      <origin xyz="0 0 0.2325" rpy="0 0 0"/>
+      <geometry>
+        <box size="0.21875 $(arg head_depth) 0.155"/>
+      </geometry>
+      <material name="head_gray"/>
+    </visual>
+    <collision>
+      <origin xyz="0 0 0.155" rpy="0 0 0"/>
+      <geometry>
+        <box size="$(arg head_upper_width) $(arg head_depth) $(arg head_height)"/>
+      </geometry>
+    </collision>
+  </link>
+  <joint name="column_to_head" type="fixed">
+    <parent link="column"/>
+    <child link="column_head"/>
+    <origin xyz="$(arg head_base_xyz)" rpy="0 0 0"/>
+  </joint>
 </robot>

Commit message: refactor(urdf): 用真实梯形mesh替换column head近似分层
- 新增精确尺寸梯形棱柱 STL（上宽0.25 下宽0.125 高0.31 厚0.125，厚度沿Y）\n- column-only 模型改为mesh visual/collision，不再使用分层box近似\n- 保持立柱中心线与顶部实体中心线重合

File: src/dual_nero_description/urdf/dual_nero_column_only.xacro (robot description, xacro)
@@ -5,9 +5,6 @@
   <xacro:arg name="column_size" default="0.105 0.105 0.52"/>
   <xacro:arg name="column_visual_xyz" default="0 0 0.26"/>
-  <xacro:arg name="head_upper_width" default="0.25"/>
-  <xacro:arg name="head_lower_width" default="0.125"/>
-  <xacro:arg name="head_depth" default="0.125"/>
-  <xacro:arg name="head_height" default="0.31"/>
   <xacro:arg name="head_base_xyz" default="0 0 0.52"/>
+  <xacro:arg name="head_mesh" default="package://dual_nero_description/meshes/generated/column_head_trapezoid.stl"/>
   <material name="column_silver">
     <color rgba="0.8 0.8 0.8 1.0"/>
@@ -39,21 +36,14 @@
   <link name="column_head">
     <visual>
-      <origin xyz="0 0 0.0775" rpy="0 0 0"/>
+      <origin xyz="0 0 0" rpy="0 0 0"/>
       <geometry>
-        <box size="0.15625 $(arg head_depth) 0.155"/>
-      </geometry>
-      <material name="head_gray"/>
-    </visual>
-    <visual>
-      <origin xyz="0 0 0.2325" rpy="0 0 0"/>
-      <geometry>
-        <box size="0.21875 $(arg head_depth) 0.155"/>
+        <mesh filename="$(arg head_mesh)"/>
       </geometry>
       <material name="head_gray"/>
     </visual>
     <collision>
-      <origin xyz="0 0 0.155" rpy="0 0 0"/>
+      <origin xyz="0 0 0" rpy="0 0 0"/>
       <geometry>
-        <box size="$(arg head_upper_width) $(arg head_depth) $(arg head_height)"/>
+        <mesh filename="$(arg head_mesh)"/>
       </geometry>
     </collision>

Commit message: feat(urdf): 在column-only模型顶部添加横杆
- 新增 top_bar 几何，尺寸为 0.255x0.02x0.02 m\n- 横杆长边沿 X 方向，与梯形顶部宽向一致\n- 横杆中心线与梯形上平面中线对齐并放置于顶部

File: src/dual_nero_description/urdf/dual_nero_column_only.xacro (robot description, xacro)
@@ -7,4 +7,6 @@
   <xacro:arg name="head_base_xyz" default="0 0 0.52"/>
   <xacro:arg name="head_mesh" default="package://dual_nero_description/meshes/generated/column_head_trapezoid.stl"/>
+  <xacro:arg name="top_bar_size" default="0.255 0.02 0.02"/>
+  <xacro:arg name="top_bar_xyz" default="0 0 0.32"/>
   <material name="column_silver">
     <color rgba="0.8 0.8 0.8 1.0"/>
@@ -54,3 +56,23 @@
     <origin xyz="$(arg head_base_xyz)" rpy="0 0 0"/>
   </joint>
+  <link name="top_bar">
+    <visual>
+      <origin xyz="0 0 0" rpy="0 0 0"/>
+      <geometry>
+        <box size="$(arg top_bar_size)"/>
+      </geometry>
+      <material name="head_gray"/>
+    </visual>
+    <collision>
+      <origin xyz="0 0 0" rpy="0 0 0"/>
+      <geometry>
+        <box size="$(arg top_bar_size)"/>
+      </geometry>
+    </collision>
+  </link>
+  <joint name="head_to_top_bar" type="fixed">
+    <parent link="column_head"/>
+    <child link="top_bar"/>
+    <origin xyz="$(arg top_bar_xyz)" rpy="0 0 0"/>
+  </joint>
 </robot>

Commit message: feat(urdf): add side white boxes on top bar with face-center alignment
- Add left/right white boxes sized 0.08x0.02x0.095 m\n- Place boxes on top bar side faces with center alignment\n- Keep box width on X so the length-height face contacts the bar side plane

File: src/dual_nero_description/urdf/dual_nero_column_only.xacro (robot description, xacro)
@@ -9,4 +9,7 @@
   <xacro:arg name="top_bar_size" default="0.255 0.02 0.02"/>
   <xacro:arg name="top_bar_xyz" default="0 0 0.32"/>
+  <xacro:arg name="side_box_size" default="0.02 0.08 0.095"/>
+  <xacro:arg name="left_side_box_xyz" default="0.1375 0 0"/>
+  <xacro:arg name="right_side_box_xyz" default="-0.1375 0 0"/>
   <material name="column_silver">
     <color rgba="0.8 0.8 0.8 1.0"/>
@@ -14,4 +17,7 @@
   <material name="head_gray">
     <color rgba="0.72 0.72 0.72 1.0"/>
+  </material>
+  <material name="box_white">
+    <color rgba="0.95 0.95 0.95 1.0"/>
   </material>
   <link name="world"/>
@@ -76,3 +82,43 @@
     <origin xyz="$(arg top_bar_xyz)" rpy="0 0 0"/>
   </joint>
+  <link name="left_side_box">
+    <visual>
+      <origin xyz="0 0 0" rpy="0 0 0"/>
+      <geometry>
+        <box size="$(arg side_box_size)"/>
+      </geometry>
+      <material name="box_white"/>
+    </visual>
+    <collision>
+      <origin xyz="0 0 0" rpy="0 0 0"/>
+      <geometry>
+        <box size="$(arg side_box_size)"/>
+      </geometry>
+    </collision>
+  </link>
+  <joint name="top_bar_to_left_side_box" type="fixed">
+    <parent link="top_bar"/>
+    <child link="left_side_box"/>
+    <origin xyz="$(arg left_side_box_xyz)" rpy="0 0 0"/>
+  </joint>
+  <link name="right_side_box">
+    <visual>
+      <origin xyz="0 0 0" rpy="0 0 0"/>
+      <geometry>
+        <box size="$(arg side_box_size)"/>
+      </geometry>
+      <material name="box_white"/>
+    </visual>
+    <collision>
+      <origin xyz="0 0 0" rpy="0 0 0"/>
+      <geometry>
+        <box size="$(arg side_box_size)"/>
+      </geometry>
+    </collision>
+  </link>
+  <joint name="top_bar_to_right_side_box" type="fixed">
+    <parent link="top_bar"/>
+    <child link="right_side_box"/>
+    <origin xyz="$(arg right_side_box_xyz)" rpy="0 0 0"/>
+  </joint>
 </robot>

Commit message: refactor(urdf): anchor dual-arm mounts to side-plate face centers
- Add left/right mount face frames at side-plate outer-face centers\n- Attach dual arms to mount-face frames instead of plate link origins\n- Keep arm offsets zero by default so alignment starts from geometric face centers

File: src/dual_nero_description/urdf/dual_nero_column_only.xacro (robot description, xacro)
@@ -14,7 +14,9 @@
   <xacro:arg name="right_side_box_xyz" default="-0.1375 0 0"/>
   <xacro:arg name="enable_arms" default="true"/>
-  <xacro:arg name="left_arm_mount_xyz" default="0.01 0 0"/>
+  <xacro:arg name="left_mount_face_xyz" default="0.01 0 0"/>
+  <xacro:arg name="right_mount_face_xyz" default="-0.01 0 0"/>
+  <xacro:arg name="left_arm_mount_xyz" default="0 0 0"/>
   <xacro:arg name="left_arm_mount_rpy" default="0 -1.5708 3.14159"/>
-  <xacro:arg name="right_arm_mount_xyz" default="-0.01 0 0"/>
+  <xacro:arg name="right_arm_mount_xyz" default="0 0 0"/>
   <xacro:arg name="right_arm_mount_rpy" default="0 -1.5708 0"/>
   <xacro:include filename="$(find dual_nero_description)/urdf/nero_single_arm_macro.xacro"/>
@@ -109,4 +111,10 @@
     <origin xyz="$(arg left_side_box_xyz)" rpy="0 0 0"/>
   </joint>
+  <link name="left_mount_face"/>
+  <joint name="left_side_box_to_mount_face" type="fixed">
+    <parent link="left_side_box"/>
+    <child link="left_mount_face"/>
+    <origin xyz="$(arg left_mount_face_xyz)" rpy="0 0 0"/>
+  </joint>
   <link name="right_side_box">
     <visual>
@@ -129,8 +137,14 @@
     <origin xyz="$(arg right_side_box_xyz)" rpy="0 0 0"/>
   </joint>
+  <link name="right_mount_face"/>
+  <joint name="right_side_box_to_mount_face" type="fixed">
+    <parent link="right_side_box"/>
+    <child link="right_mount_face"/>
+    <origin xyz="$(arg right_mount_face_xyz)" rpy="0 0 0"/>
+  </joint>
   <xacro:if value="$(arg enable_arms)">
     <xacro:nero_single_arm
         prefix="left_"
-        parent="left_side_box"
+        parent="left_mount_face"
         xyz="$(arg left_arm_mount_xyz)"
         rpy="$(arg left_arm_mount_rpy)"
@@ -138,5 +152,5 @@
     <xacro:nero_single_arm
         prefix="right_"
-        parent="right_side_box"
+        parent="right_mount_face"
         xyz="$(arg right_arm_mount_xyz)"
         rpy="$(arg right_arm_mount_rpy)"
