Commit message: fix(sim): 修复 xacro 弃用警告导致的仿真启动失败
- 将 ros2_control xacro 中的 load_yaml() 切换为 xacro.load_yaml()\n- 避免 simulation.launch.py 在生成 robot_description 时因 stderr 警告被 launch 误判为失败

File: src/dual_nero_moveit_config/config/dual_nero_description.ros2_control.xacro (robot description, xacro)
@@ -5,5 +5,5 @@
         params="name initial_positions_file hardware_plugin:='mock_components/GenericSystem' use_gz_sim:='false' controllers_file:=''"
     >
-        <xacro:property name="initial_positions" value="${load_yaml(initial_positions_file)['initial_positions']}"/>
+        <xacro:property name="initial_positions" value="${xacro.load_yaml(initial_positions_file)['initial_positions']}"/>
         <ros2_control name="${name}" type="system">
             <hardware>

Commit message: fix(sim): 修复 gz_ros2_control 插件生成条件
- 将 ros2_control xacro 中的 use_gz_sim 判断改为兼容字符串/布尔的稳妥形式\n- 确保 use_gz_sim=true 时 GazeboSimROS2ControlPlugin 真正生成进 URDF\n- 为 controller_manager、joint_states 和仿真 FollowJointTrajectory 控制链恢复提供前提

File: src/dual_nero_moveit_config/config/dual_nero_description.ros2_control.xacro (robot description, xacro)
@@ -6,4 +6,5 @@
     >
         <xacro:property name="initial_positions" value="${xacro.load_yaml(initial_positions_file)['initial_positions']}"/>
+        <xacro:property name="gz_sim_enabled" value="${str(use_gz_sim).lower() == 'true'}"/>
         <ros2_control name="${name}" type="system">
             <hardware>
@@ -109,5 +110,5 @@
             </joint>
         </ros2_control>
-        <xacro:if value="${use_gz_sim == 'true'}">
+        <xacro:if value="${gz_sim_enabled}">
             <gazebo>
                 <plugin filename="libgz_ros2_control-system.so" name="gz_ros2_control::GazeboSimROS2ControlPlugin">
